File: converter-30-plus-10-pin/pcb/framework-laptop-converter.kicad_pcb (KiCad board)
At the start: 4 copper layers, 20 x 40 mm, 7 parts, among them J1 20455-040E-76, J2 FFC2B28-40-G

Commit message: for some reason these are backwards too
Connections:
- J1 pad 32: BL_EN -> (no net)
Routing:
- net BL_EN: track 38.5 -> 0.00 mm
- net EDP_AUX_P: track 37.7 -> 7.16 mm
- net EDP_AUX_N: track 37.7 -> 7.16 mm
- net EDP_HPD: track 37.9 -> 7.98 mm
- net EDP_SELF_TEST: track 38.2 -> 10.1 mm
- net BL_PWM_DIM: track 39.3 -> 12.9 mm
- net EDP_LANE0_P: track 33.5 -> 7.16 mm
- net EDP_LANE0_N: track 33.4 -> 7.16 mm
- net EDP_LANE1_P: track 26.2 -> 7.16 mm
- net EDP_LANE1_N: track 26.1 -> 7.16 mm
- net GND: vias 2 -> 0
