File: breakout/pcb/framework-laptop-edp-breakout.kicad_pcb (KiCad board)
At the start: 2 copper layers, 29 x 46 mm, 6 parts, among them J1 20879-040E-01, J2 Conn_01x40

Commit message: add revision to the breakout because I'm losing track
Other:
- board text added: "Framework Laptop I-PEX 20879-040E Breakout for eDP / Touchscreen v${REVISION}"
- board text removed: "Framework Laptop I-PEX 20879-040E Breakout for eDP / Touchscreen"
Changed lines of the file:
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@@
   (gr_arc (start 153.99998 56) (mid 154.878661 53.878687) (end 156.99998 53) (layer "Edge.Cuts") (width 0.1))
   (gr_line (start 183 56) (end 183 96) (layer "Edge.Cuts") (width 0.1))
-  (gr_text "Framework Laptop\nI-PEX 20879-040E Breakout\nfor eDP / Touchscreen\n" (at 160.782 75.819 90) (layer "B.SilkS")
+  (gr_text "Framework Laptop\nI-PEX 20879-040E Breakout\nfor eDP / Touchscreen\n\nv${REVISION}" (at 162.2 76 90) (layer "B.SilkS")
     (effects (font (size 1 1) (thickness 0.15)) (justify mirror))
   )
@@
   (zone (net 15) (net_name "EDP_3V") (layer "F.Cu") (hatch edge 0.508)
     (priority 1)
-    (connect_pads (clearance 0.2))
+    (connect_pads yes (clearance 0.2))
     (min_thickness 0.15) (filled_areas_thickness no)
     (fill yes (thermal_gap 0.15) (thermal_bridge_width 0.15) (island_removal_mode 1) (island_area_min 0))
@@
   (zone (net 16) (net_name "BL_POWER") (layer "F.Cu") (hatch edge 0.508)
     (priority 1)
-    (connect_pads (clearance 0.2))
+    (connect_pads yes (clearance 0.2))
     (min_thickness 0.15) (filled_areas_thickness no)
     (fill yes (thermal_gap 0.15) (thermal_bridge_width 0.15) (island_removal_mode 1) (island_area_min 0))
@@
   (zone (net 15) (net_name "EDP_3V") (layer "B.Cu") (hatch edge 0.508)
     (priority 1)
-    (connect_pads (clearance 0.2))
+    (connect_pads yes (clearance 0.2))
     (min_thickness 0.15) (filled_areas_thickness no)
     (fill yes (thermal_gap 0.15) (thermal_bridge_width 0.5) (island_removal_mode 1) (island_area_min 0))
@@
   (zone (net 16) (net_name "BL_POWER") (layer "B.Cu") (hatch edge 0.508)
     (priority 1)
-    (connect_pads (clearance 0.2))
+    (connect_pads yes (clearance 0.2))
     (min_thickness 0.254) (filled_areas_thickness no)
     (fill yes (thermal_gap 0.508) (thermal_bridge_width 0.508))
